File: PCB_SHEMS/ESP_Edgedevice/ESP_Edgedevice.kicad_pcb (KiCad board)
At the start: 2 copper layers, 125 x 100 mm, 57 parts, among them J1 Barrier Terminal, J2 HB9500-9.5-3P, J3 Conn_01x02_Pin, J4 Conn_01x02, K1 SLA-05VDC-SL-C, Q1 S8050, U1 XIAO ESP32C3, U2 PC817X3NSZ1B, U3 AMS1117-5.0, U4 AMC1200SDUBR, U5 OPA333xxDBV, U6 OPA333xxDBV, U7 MCP3202

Commit message: started PCB
Parts:
- C10, C11, C13, C14, C15, C8: footprint Capacitor_THT:C_Disc_D5.0mm_W2.5mm_P5.00mm -> Capacitor_SMD:C_1206_3216Metric
- C16, C9: footprint Capacitor_SMD:C_0805_2012Metric -> Capacitor_SMD:C_1206_3216Metric
- C5: footprint Capacitor_THT:CP_Radial_D10.0mm_P5.00mm -> Capacitor_SMD:C_1206_3216Metric
- C6: footprint Capacitor_THT:C_Disc_D5.0mm_W2.5mm_P5.00mm -> Capacitor_THT:CP_Radial_D5.0mm_P2.50mm
- J2: footprint Connector_Phoenix_MSTB:PhoenixContact_MSTBA_2,5_3-G_1x03_P5.00mm_Horizontal -> myparts:HB9500_9.5-3P
- R1, R10, R11, R12, R13, R14, R15, R16, R3, R8, R9: footprint Resistor_THT:R_Axial_DIN0207_L6.3mm_D2.5mm_P10.16mm_Horizontal -> Resistor_SMD:R_1206_3216Metric
- R2: value 2.2K -> 1k; footprint Resistor_THT:R_Axial_DIN0207_L6.3mm_D2.5mm_P10.16mm_Horizontal -> Resistor_SMD:R_1206_3216Metric
- U1: footprint xiao-esp32-c3:xiao_esp32c3 -> myparts:XIAO_Socket_W15.24
- U7: footprint Package_SO:TSSOP-8_3x3mm_P0.65mm -> Package_SO:TSSOP-8_4.4x3mm_P0.65mm
Other:
- outline, holes or cut-outs redrawn

Commit message: 2nd ADS
Parts:
- added C10: 100nF, Capacitor_SMD:C_1206_3216Metric, F.Cu at (87.3, 124.5)
- added C11: 100nF, Capacitor_SMD:C_1206_3216Metric, F.Cu at (87.3, 127.9)
- added C12: 100nF, Capacitor_SMD:C_1206_3216Metric, F.Cu at (87.3, 131.2)
- added C13: 100nF, Capacitor_SMD:C_1206_3216Metric, F.Cu at (87.3, 134.6)
- added C9: 100nF, Capacitor_SMD:C_1206_3216Metric, F.Cu at (87.3, 121.2)
- added D5: D_TVS, Diode_SMD:Nexperia_DSN0603-2_0.6x0.3mm_P0.4mm, F.Cu at (96.4, 135.4)
- added R12: 0.33 Ω, 1206, Resistor_SMD:R_1206_3216Metric, F.Cu at (101.7, 131.6)
- added R18: 1k, Resistor_SMD:R_1206_3216Metric, F.Cu at (101.7, 134.9)
- added U6: OPA333xxDBV, Package_TO_SOT_SMD:SOT-23-5, F.Cu at (92.7, 136.9)
- added U7: MCP3202, Package_SO:TSSOP-8_4.4x3mm_P0.65mm, F.Cu at (94.5, 132.3)
- added U8: AMC1200SDUBR, AMC1200SDUBR:DUB0008A-IPC_A, F.Cu at (97.3, 124.7)
- moved J2 16.9 mm to (121.0, 116.2)
Connections:
- J4 pad 1: /voltagesensing.kicad_sch/VBIAS_BUF -> Net-(D5-A1)
- J4 pad 2: Net-(J4-Pin_2) -> GND
- R15 pad 2: Net-(U7-CH0) -> /voltagesensing.kicad_sch/V_ADC

Commit message: changes
Parts:
- moved H3 84.7 mm to (200.0, 137.5)
- moved H4 83.1 mm to (85.0, 137.5)
- moved H2 74.5 mm to (200.0, 47.5)
- moved H1 54.9 mm to (85.0, 47.5)
- moved J2 18.0 mm to (136.0, 126.2)
- moved U8 17.8 mm to (115.0, 122.5)
- moved C10 17.3 mm to (104.5, 123.5)
- moved C11 17.3 mm to (104.5, 126.8)
- moved C12 17.3 mm to (104.5, 130.2)
- moved C13 17.3 mm to (104.5, 133.5)
- moved C9 17.3 mm to (104.5, 120.1)
- moved D5 17.3 mm to (113.6, 134.3)
- moved R12 17.3 mm to (118.9, 130.6)
- moved R18 17.3 mm to (118.9, 133.9)
- moved U6 17.3 mm to (109.9, 135.9)
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Changed lines of the file:
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@@
 	(footprint "Package_TO_SOT_SMD:SOT-23-5"
 		(layer "F.Cu")
-		(at 92.725 136.93)
+		(at 109.948112 135.9025)
 		(descr "SOT, 5 Pin (JEDEC MO-178 Var AA https://www.jedec.org/document_search?search_api_views_fulltext=MO-178)")
 		(tags "SOT TO_SOT_SMD")
@@
 	(footprint "MountingHole:MountingHole_2.1mm"
 		(layer "F.Cu")
-		(at 132.925 80.025)
+		(at 200 47.5)
 		(descr "Mounting Hole 2.1mm, no annular, generated by kicad-footprint-generator mountinghole.py")
 		(tags "mountinghole")
@@
 		)
 		(property "Value" "25A Slow-Blow"
-			(at 18.95 8.8 0)
+			(at 19.225 4.725 0)
 			(layer "F.Fab")
 			(effects
@@
 	(footprint "myparts:XIAO_Socket_W15.24"
 		(layer "F.Cu")
-		(at 99.5 102.325)
+		(at 99.5 102.325 90)
 		(descr "14-lead though-hole mounted DIP package, row spacing 10.16mm (400 mils)")
 		(tags "THT DIP DIL PDIP 2.54mm 10.16mm 400mil")
 		(property "Reference" "U1"
-			(at 0.525 -10.45 0)
+			(at 0.525 -10.45 90)
 			(layer "F.SilkS")
 			(effects
@@
 		)
 		(property "Value" "XIAO ESP32C3"
-			(at -0.3025 9.88 0)
+			(at -0.3025 9.88 90)
 			(layer "F.Fab")
 			(effects
@@
 		)
 		(property "Datasheet" "https://files.seeedstudio.com/wiki/Seeed-Studio-XIAO-ESP32/esp32-c3_datasheet.pdf"
-			(at 0 0 0)
+			(at 0 0 90)
 			(layer "F.Fab")
 			(hide yes)
@@
 		)
 		(property "Description" "ESP32C3 Transceiver Evaluation Board"
-			(at 0 0 0)
+			(at 0 0 90)
 			(layer "F.Fab")
 			(hide yes)
@@
 		)
 		(property "KiLib_Generator" "package/DIP/legacy"
-			(at 0 0 0)
+			(at 0 0 90)
 			(layer "F.SilkS")
 			(hide yes)
@@
 		)
 		(property "MANUFACTURER" "Seeed Technology"
-			(at 0 0 0)
+			(at 0 0 90)
 			(unlocked yes)
 			(layer "F.Fab")
@@
 		(duplicate_pad_numbers_are_jumpers no)
 		(fp_line
-			(start -6.13 -9.45)
-			(end -6.13 8.45)
+			(start 5.6425 -9.45)
+			(end 3.4075 -9.45)
 			(stroke
 				(width 0.12)
@@
 		)
 		(fp_line
-			(start -6.13 8.45)
-			(end 5.525 8.45)
+			(start -3.895 -9.45)
+			(end -6.13 -9.45)
 			(stroke
 				(width 0.12)
@@
 		)
 		(fp_line
-			(start -3.895 -9.45)
-			(end -6.13 -9.45)
+			(start -6.13 -9.45)
+			(end -6.13 8.45)
 			(stroke
 				(width 0.12)
@@
 		)
 		(fp_line
-			(start 5.6425 -9.45)
-			(end 3.4075 -9.45)
+			(start -6.13 8.45)
+			(end 5.525 8.45)
 			(stroke
 				(width 0.12)
@@
 		)
 		(fp_line
-			(start -6.07 -8.39)
-			(end -5.07 -9.39)
+			(start 5.36 -9.39)
+			(end 5.36 8.39)
 			(stroke
 				(width 0.1)
@@
 		)
 		(fp_line
-			(start -6.07 8.39)
-			(end -6.07 -8.39)
+			(start -5.07 -9.39)
+			(end 4.025 -9.39)
 			(stroke
 				(width 0.1)
@@
 		)
 		(fp_line
-			(start -5.07 -9.39)
-			(end 4.025 -9.39)
+			(start -6.07 -8.39)
+			(end -5.07 -9.39)
 			(stroke
 				(width 0.1)
@@
 		)
 		(fp_line
-			(start 0.28 8.39)
-			(end -6.07 8.39)
+			(start 5.525 -8.12)
+			(end 4.525 -9.12)
 			(stroke
 				(width 0.1)
@@
 		)
 		(fp_line
-			(start 5.36 -9.39)
-			(end 5.36 8.39)
+			(start 0.28 8.39)
+			(end -6.07 8.39)
 			(stroke
 				(width 0.1)
@@
 		)
 		(fp_line
-			(start 5.525 -8.12)
-			(end 4.525 -9.12)
+			(start -6.07 8.39)
+			(end -6.07 -8.39)
 			(stroke
 				(width 0.1)
@@
 		)
 		(fp_text user "${REFERENCE}"
-			(at 0.025 -0.5 90)
+			(at 0.025 -0.5 0)
 			(layer "F.Fab")
 			(effects
@@
 		)
 		(point
-			(at 99.525 101.825)
+			(at 99 102.3)
 			(size 1.27)
 			(layer "F.Fab")
 		)
 		(pad "1" thru_hole roundrect
-			(at -7.975 -8.12)
+			(at -7.975 -8.12 90)
 			(size 1.6 1.6)
 			(drill 0.8)
@@
 		)
 		(pad "2" thru_hole circle
-			(at -7.975 -5.58)
+			(at -7.975 -5.58 90)
 			(size 1.6 1.6)
 			(drill 0.8)
@@
 		)
 		(pad "3" thru_hole circle
-			(at -7.975 -3.04)
+			(at -7.975 -3.04 90)
 			(size 1.6 1.6)
 			(drill 0.8)
@@
 		)
 		(pad "4" thru_hole circle
-			(at -7.975 -0.5)
+			(at -7.975 -0.5 90)
 			(size 1.6 1.6)
 			(drill 0.8)
@@
 		)
 		(pad "5" thru_hole circle
-			(at -7.975 2.04)
+			(at -7.975 2.04 90)
 			(size 1.6 1.6)
 			(drill 0.8)
@@
 		)
 		(pad "6" thru_hole circle
-			(at -7.975 4.58)
+			(at -7.975 4.58 90)
 			(size 1.6 1.6)
 			(drill 0.8)
@@
 		)
 		(pad "7" thru_hole circle
-			(at -7.975 7.12)
+			(at -7.975 7.12 90)
 			(size 1.6 1.6)
 			(drill 0.8)
@@
 		)
 		(pad "8" thru_hole circle
-			(at 7.265 7.12)
+			(at 7.265 7.12 90)
 			(size 1.6 1.6)
 			(drill 0.8)
@@
 		)
 		(pad "9" thru_hole circle
-			(at 7.265 4.58)
+			(at 7.265 4.58 90)
 			(size 1.6 1.6)
 			(drill 0.8)
@@
 		)
 		(pad "10" thru_hole circle
-			(at 7.265 2.04)
+			(at 7.265 2.04 90)
 			(size 1.6 1.6)
 			(drill 0.8)
@@
 		)
 		(pad "11" thru_hole circle
-			(at 7.265 -0.5)
+			(at 7.265 -0.5 90)
 			(size 1.6 1.6)
 			(drill 0.8)
@@
 		)
 		(pad "12" thru_hole circle
-			(at 7.265 -3.04)
+			(at 7.265 -3.04 90)
 			(size 1.6 1.6)
 			(drill 0.8)
@@
 		)
 		(pad "13" thru_hole circle
-			(at 7.265 -5.58)
+			(at 7.265 -5.58 90)
 			(size 1.6 1.6)
 			(drill 0.8)
@@
 		)
 		(pad "14" thru_hole circle
-			(at 7.265 -8.12)
+			(at 7.265 -8.12 90)
 			(size 1.6 1.6)
 			(drill 0.8)
@@
 	(footprint "AMC1200SDUBR:DUB0008A-IPC_A"
 		(layer "F.Cu")
-		(at 97.302076 124.7175)
+		(at 115 122.5)
 		(tags "AMC1200SDUBR ")
 		(property "Reference" "U8"
@@
 	(footprint "Capacitor_SMD:C_1206_3216Metric"
 		(layer "F.Cu")
-		(at 87.325 131.225)
+		(at 104.548112 130.1975)
 		(descr "Capacitor SMD 1206 (3216 Metric), square (rectangular) end terminal, IPC-7351 nominal, (Body size source: IPC-SM-782 page 76, https://www.pcb-3d.com/wordpress/wp-content/uploads/ipc-sm-782a_amendment_1_and_2.pdf)")
 		(tags "capacitor")
@@
 	(footprint "Resistor_SMD:R_1206_3216Metric"
 		(layer "F.Cu")
-		(at 101.705 131.585)
+		(at 118.928112 130.5575)
 		(descr "Resistor SMD 1206 (3216 Metric), square (rectangular) end terminal, IPC-7351 nominal, (Body size source: IPC-SM-782 page 72, https://www.pcb-3d.com/wordpress/wp-content/uploads/ipc-sm-782a_amendment_1_and_2.pdf)")
 		(tags "resistor")
@@
 	(footprint "MountingHole:MountingHole_2.1mm"
 		(layer "F.Cu")
-		(at 132.925 85.775)
+		(at 200 137.5)
 		(descr "Mounting Hole 2.1mm, no annular, generated by kicad-footprint-generator mountinghole.py")
 		(tags "mountinghole")
@@
 	(footprint "Resistor_SMD:R_1206_3216Metric"
 		(layer "F.Cu")
-		(at 101.705 134.895)
+		(at 118.928112 133.8675)
 		(descr "Resistor SMD 1206 (3216 Metric), square (rectangular) end terminal, IPC-7351 nominal, (Body size source: IPC-SM-782 page 72, https://www.pcb-3d.com/wordpress/wp-content/uploads/ipc-sm-782a_amendment_1_and_2.pdf)")
 		(tags "resistor")
@@
 	(footprint "Diode_SMD:Nexperia_DSN0603-2_0.6x0.3mm_P0.4mm"
 		(layer "F.Cu")
-		(at 96.42 135.355)
+		(at 113.643112 134.3275)
 		(descr "SOD962-2 silicon, leadless ultra small package; 2 terminals; 0.4 mm pitch; 0.6 mm x 0.3 mm x 0.3 mm body (https://assets.nexperia.com/documents/package-information/SOD962-2.pdf https://www.nexperia.com/packages/SOD962-2.html)")
 		(tags "TVS protection diodes")
@@
 	(footprint "Capacitor_SMD:C_1206_3216Metric"
 		(layer "F.Cu")
-		(at 87.325 134.575)
+		(at 104.548112 133.5475)
 		(descr "Capacitor SMD 1206 (3216 Metric), square (rectangular) end terminal, IPC-7351 nominal, (Body size source: IPC-SM-782 page 76, https://www.pcb-3d.com/wordpress/wp-content/uploads/ipc-sm-782a_amendment_1_and_2.pdf)")
 		(tags "capacitor")
@@
 	(footprint "MountingHole:MountingHole_2.1mm"
 		(layer "F.Cu")
-		(at 132.925 74.275)
+		(at 85 47.5)
 		(descr "Mounting Hole 2.1mm, no annular, generated by kicad-footprint-generator mountinghole.py")
 		(tags "mountinghole")
@@
 	(footprint "Capacitor_SMD:C_1206_3216Metric"
 		(layer "F.Cu")
-		(at 87.325 124.525)
+		(at 104.548112 123.4975)
 		(descr "Capacitor SMD 1206 (3216 Metric), square (rectangular) end terminal, IPC-7351 nominal, (Body size source: IPC-SM-782 page 76, https://www.pcb-3d.com/wordpress/wp-content/uploads/ipc-sm-782a_amendment_1_and_2.pdf)")
 		(tags "capacitor")
@@
 		(tags "ACDC-Converter 5W THT Hi-Link board mount module")
 		(property "Reference" "PS1"
-			(at 16.8 -10.7 0)
+			(at 16.8 -6.575 0)
 			(layer "F.SilkS")
 			(effects
@@
 	(footprint "myparts:HB9500_9.5-3P"
 		(layer "F.Cu")
-		(at 121 116.2225)
+		(at 136 126.2225)
 		(descr "Generic Phoenix Contact connector footprint for: MSTBA_2,5/3-G; number of pins: 03; pin pitch: 5.00mm; Angled || order number: 1757488 12A || order number: 1923762 16A (HC)")
 		(tags "phoenix_contact connector MSTBA_01x03_G_5.00mm")
@@
 	(footprint "Capacitor_SMD:C_1206_3216Metric"
 		(layer "F.Cu")
-		(at 87.325 127.875)
+		(at 104.548112 126.8475)
 		(descr "Capacitor SMD 1206 (3216 Metric), square (rectangular) end terminal, IPC-7351 nominal, (Body size source: IPC-SM-782 page 76, https://www.pcb-3d.com/wordpress/wp-content/uploads/ipc-sm-782a_amendment_1_and_2.pdf)")
 		(tags "capacitor")
@@
 	(footprint "MountingHole:MountingHole_2.1mm"
 		(layer "F.Cu")
-		(at 142.375 77.375)
+		(at 85 137.5)
 		(descr "Mounting Hole 2.1mm, no annular, generated by kicad-footprint-generator mountinghole.py")
 		(tags "mountinghole")
@@
 	(footprint "Package_SO:TSSOP-8_4.4x3mm_P0.65mm"
 		(layer "F.Cu")
-		(at 94.525 132.26)
+		(at 111.748112 131.2325)
 		(descr "TSSOP, 8 Pin (JEDEC MO-153 Var AA https://www.jedec.org/document_search?search_api_views_fulltext=MO-153)")
 		(tags "TSSOP SO")
@@
 	(footprint "Capacitor_SMD:C_1206_3216Metric"
 		(layer "F.Cu")
-		(at 87.325 121.175)
+		(at 104.548112 120.1475)
 		(descr "Capacitor SMD 1206 (3216 Metric), square (rectangular) end terminal, IPC-7351 nominal, (Body size source: IPC-SM-782 page 76, https://www.pcb-3d.com/wordpress/wp-content/uploads/ipc-sm-782a_amendment_1_and_2.pdf)")
 		(tags "capacitor")
